Commit message: add circle stacks

File: create2_description/urdf/common_properties.urdf.xacro (robot description, xacro)
@@ -3,5 +3,5 @@
   Various useful properties such as constants and materials
  -->
-<root name="xacro_properties" xmlns:xacro="http://www.ros.org/wiki/xacro">
+<robot name="xacro_properties" xmlns:xacro="http://ros.org/wiki/xacro">
   <xacro:property name="M_PI" value="3.1415926535897931" />
   <xacro:property name="material_white">
@@ -55,3 +55,3 @@
     </material>
   </xacro:property>
-</root>
+</robot>

File: create2_description/urdf/create2/create_base.urdf.xacro (robot description, xacro)
@@ -30,5 +30,5 @@
   </xacro:macro>
   <xacro:macro name="create_base" params="diffdrive_update_rate:=40 wheel_separation wheel_radius:=0.036 wheel_width:=0.024 wheel_torque:=1.0 wheel_accel:=1.8 mass_kg:=3.5 base_diameter *mesh">
-    <xacro:include filename="$(find create2_description)/urdf/create_base_gazebo.urdf.xacro" />
+    <xacro:include filename="$(find create2_description)/urdf/create2/create_base_gazebo.urdf.xacro" />
     <link name="base_footprint">
     <visual>

File: create2_description/urdf/sensors/kinect_properties.urdf.xacro (robot description, xacro)
@@ -4,7 +4,8 @@
 	  Translation and rotation of camera from its base link
    -->
-	<property name="cam_px" value="0" />
-	<property name="cam_py" value="0" />
-	<property name="cam_pz" value="0.1" />
+	<property name="cam_px" value="-0.087" />
+	<property name="cam_py" value="-0.0125" />
+	<!-- Y varies for different configurations. get sets in sensors_urdf  -->
+	<property name="cam_pz" value="0.17" />
 	<property name="cam_or" value="0" />
 	<property name="cam_op" value="0" />

File: create2_description/urdf/stacks/circles.urdf.xacro (robot description, xacro)
@@ -1,5 +1,5 @@
 <?xml version="1.0"?>
-<robot name="turtlebot_hardware" xmlns:xacro="http://ros.org/wiki/xacro">
-  <xacro:macro name="turtlebot_spacer" params="parent number x_loc y_loc z_loc">
+<robot name="create2_hardware" xmlns:xacro="http://ros.org/wiki/xacro">
+  <xacro:macro name="create2_spacer" params="parent number x_loc y_loc z_loc">
     <joint name="spacer_${number}_joint" type="fixed">
       <origin xyz="${x_loc} ${y_loc} ${z_loc}" rpy="0 0 0" />
@@ -18,5 +18,5 @@
         <origin xyz=" 0 0 0 " rpy="0 0 0" />
         <geometry>
-          <mesh filename="package://turtlebot_description/meshes/stacks/circles/68-02403-125_Spacer.dae"/>
+          <mesh filename="package://create2_description/meshes/stacks/circles/68-02403-125_Spacer.dae"/>
         </geometry>
       </visual>
@@ -29,5 +29,5 @@
     </link>
   </xacro:macro>
-  <xacro:macro name="turtlebot_standoff_1in" params="parent number x_loc y_loc z_loc">
+  <xacro:macro name="create2_standoff_1in" params="parent number x_loc y_loc z_loc">
     <joint name="standoff_1in_${number}_joint" type="fixed">
       <origin xyz="${x_loc} ${y_loc} ${z_loc}" rpy="0 0 0" />
@@ -46,5 +46,5 @@
         <origin xyz=" 0 0 0 " rpy="0 0 0" />
         <geometry>
-          <mesh filename="package://turtlebot_description/meshes/stacks/circles/68-04552-1000-RA_Turtlebot_M-F_Standoff.dae"/>
+          <mesh filename="package://create2_description/meshes/stacks/circles/68-04552-1000-RA_Turtlebot_M-F_Standoff.dae"/>
         </geometry>
       </visual>
@@ -57,5 +57,5 @@
     </link>
   </xacro:macro>
-  <xacro:macro name="turtlebot_standoff_2in" params="parent number x_loc y_loc z_loc">
+  <xacro:macro name="create2_standoff_2in" params="parent number x_loc y_loc z_loc">
     <joint name="standoff_2in_${number}_joint" type="fixed">
       <origin xyz="${x_loc} ${y_loc} ${z_loc}" rpy="0 0 0" />
@@ -74,5 +74,5 @@
         <origin xyz=" 0 0 0 " rpy="0 0 0" />
         <geometry>
-          <mesh filename="package://turtlebot_description/meshes/stacks/circles/68-04552-2000-RA_Turtlebot_M-F_Standoff.dae"/>
+          <mesh filename="package://create2_description/meshes/stacks/circles/68-04552-2000-RA_Turtlebot_M-F_Standoff.dae"/>
         </geometry>
       </visual>
@@ -85,5 +85,5 @@
     </link>
   </xacro:macro>
-  <xacro:macro name="turtlebot_standoff_8in" params="parent number x_loc y_loc z_loc">
+  <xacro:macro name="create2_standoff_8in" params="parent number x_loc y_loc z_loc">
     <joint name="standoff_8in_${number}_joint" type="fixed">
       <origin xyz="${x_loc} ${y_loc} ${z_loc}" rpy="0 0 0" />
@@ -102,5 +102,5 @@
         <origin xyz=" 0 0 0 " rpy="0 0 0" />
         <geometry>
-          <mesh filename="package://turtlebot_description/meshes/stacks/circles/68-02421-8000-RA_Turtlebot_F-F_Standoff.dae"/>
+          <mesh filename="package://create2_description/meshes/stacks/circles/68-02421-8000-RA_Turtlebot_F-F_Standoff.dae"/>
         </geometry>
       </visual>
@@ -113,5 +113,5 @@
     </link>
   </xacro:macro>
-  <xacro:macro name="turtlebot_standoff_kinect" params="parent number x_loc y_loc z_loc">
+  <xacro:macro name="create2_standoff_kinect" params="parent number x_loc y_loc z_loc">
     <joint name="standoff_kinect_${number}_joint" type="fixed">
       <origin xyz="${x_loc} ${y_loc} ${z_loc}" rpy="0 0 0" />
@@ -130,5 +130,5 @@
         <origin xyz=" 0 0 0 " rpy="0 0 0" />
         <geometry>
-          <mesh filename="package://turtlebot_description/meshes/stacks/circles/68-04556-RA_Kinect_Standoff_Assy.dae"/>
+          <mesh filename="package://create2_description/meshes/stacks/circles/68-04556-RA_Kinect_Standoff_Assy.dae"/>
         </geometry>
       </visual>
@@ -142,8 +142,8 @@
   </xacro:macro>
   <xacro:macro name="stack_circles" params="parent">
-    <turtlebot_spacer parent="${parent}" number="0" x_loc="-0.00254" y_loc="0.1114679" z_loc="0.062992"/>
-    <turtlebot_spacer parent="${parent}" number="1" x_loc="-0.00254" y_loc="-0.1114679" z_loc="0.062992"/>
-    <turtlebot_spacer parent="${parent}" number="2" x_loc="-0.07239" y_loc="-0.1114679" z_loc="0.062992"/>
-    <turtlebot_spacer parent="${parent}" number="3" x_loc="-0.07239" y_loc="0.1114679" z_loc="0.062992"/>
+    <create2_spacer parent="${parent}" number="0" x_loc="-0.00254" y_loc="0.1114679" z_loc="0.062992"/>
+    <create2_spacer parent="${parent}" number="1" x_loc="-0.00254" y_loc="-0.1114679" z_loc="0.062992"/>
+    <create2_spacer parent="${parent}" number="2" x_loc="-0.07239" y_loc="-0.1114679" z_loc="0.062992"/>
+    <create2_spacer parent="${parent}" number="3" x_loc="-0.07239" y_loc="0.1114679" z_loc="0.062992"/>
     <joint name="plate_0_joint" type="fixed">
       <origin xyz="-0.04334 0  0.06775704" rpy="0 0 0" />
@@ -162,5 +162,5 @@
         <origin xyz=" 0 0 0 " rpy="0 0 0" />
         <geometry>
-          <mesh filename="package://turtlebot_description/meshes/stacks/circles/plate_0_logo.dae"/>
+          <mesh filename="package://create2_description/meshes/stacks/circles/plate_0_logo.dae"/>
         </geometry>
       </visual>
@@ -172,8 +172,8 @@
       </collision>
     </link>
-    <turtlebot_standoff_2in parent="${parent}" number="0" x_loc="0.0676402" y_loc="0.1314196" z_loc="0.0709803"/>
-    <turtlebot_standoff_2in parent="${parent}" number="1" x_loc="0.0676402" y_loc="-0.1314196" z_loc="0.0709803"/>
-    <turtlebot_standoff_2in parent="${parent}" number="2" x_loc="-0.052832" y_loc="-0.1314196" z_loc="0.0709803"/>
-    <turtlebot_standoff_2in parent="${parent}" number="3" x_loc="-0.052832" y_loc="0.1314196" z_loc="0.0709803"/>
+    <create2_standoff_2in parent="${parent}" number="0" x_loc="0.0676402" y_loc="0.1314196" z_loc="0.0709803"/>
+    <create2_standoff_2in parent="${parent}" number="1" x_loc="0.0676402" y_loc="-0.1314196" z_loc="0.0709803"/>
+    <create2_standoff_2in parent="${parent}" number="2" x_loc="-0.052832" y_loc="-0.1314196" z_loc="0.0709803"/>
+    <create2_standoff_2in parent="${parent}" number="3" x_loc="-0.052832" y_loc="0.1314196" z_loc="0.0709803"/>
     <joint name="plate_1_joint" type="fixed">
       <origin xyz="0.04068 0 0.05715" rpy="0 0 0" />
@@ -192,5 +192,5 @@
         <origin xyz=" 0 0 0 " rpy="0 0 0" />
         <geometry>
-          <mesh filename="package://turtlebot_description/meshes/stacks/circles/plate_1_logo.dae"/>
+          <mesh filename="package://create2_description/meshes/stacks/circles/plate_1_logo.dae"/>
         </geometry>
       </visual>
@@ -202,8 +202,8 @@
       </collision>
     </link>
-    <turtlebot_standoff_2in parent="standoff_2in_0_link" number="4" x_loc="0" y_loc="0" z_loc="0.05715"/>
-    <turtlebot_standoff_2in parent="standoff_2in_1_link" number="5" x_loc="0" y_loc="0" z_loc="0.05715"/>
-    <turtlebot_standoff_2in parent="standoff_2in_2_link" number="6" x_loc="0" y_loc="0" z_loc="0.05715"/>
-    <turtlebot_standoff_2in parent="standoff_2in_3_link" number="7" x_loc="0" y_loc="0" z_loc="0.05715"/>
+    <create2_standoff_2in parent="standoff_2in_0_link" number="4" x_loc="0" y_loc="0" z_loc="0.05715"/>
+    <create2_standoff_2in parent="standoff_2in_1_link" number="5" x_loc="0" y_loc="0" z_loc="0.05715"/>
+    <create2_standoff_2in parent="standoff_2in_2_link" number="6" x_loc="0" y_loc="0" z_loc="0.05715"/>
+    <create2_standoff_2in parent="standoff_2in_3_link" number="7" x_loc="0" y_loc="0" z_loc="0.05715"/>
     <joint name="plate_2_joint" type="fixed">
       <origin xyz="0 0 0.0572008" rpy="0 0 0" />
@@ -222,5 +222,5 @@
         <origin xyz=" 0 0 0 " rpy="0 0 0" />
         <geometry>
-          <mesh filename="package://turtlebot_description/meshes/stacks/circles/plate_1_logo.dae"/>
+          <mesh filename="package://create2_description/meshes/stacks/circles/plate_1_logo.dae"/>
         </geometry>
       </visual>
@@ -232,10 +232,10 @@
       </collision>
     </link>
-    <turtlebot_standoff_kinect parent="plate_2_link" number="0" x_loc="-0.1024382" y_loc="0.098" z_loc="0.0032004"/>
-    <turtlebot_standoff_kinect parent="plate_2_link" number="1" x_loc="-0.1024382" y_loc="-0.098" z_loc="0.0032004"/>
-    <turtlebot_standoff_8in parent="standoff_2in_4_link" number="0" x_loc="0" y_loc="0" z_loc="0.05715"/>
-    <turtlebot_standoff_8in parent="standoff_2in_5_link" number="1" x_loc="0" y_loc="0" z_loc="0.05715"/>
-    <turtlebot_standoff_8in parent="standoff_2in_6_link" number="2" x_loc="0" y_loc="0" z_loc="0.05715"/>
-    <turtlebot_standoff_8in parent="standoff_2in_7_link" number="3" x_loc="0" y_loc="0" z_loc="0.05715"/>
+    <create2_standoff_kinect parent="plate_2_link" number="0" x_loc="-0.1024382" y_loc="0.098" z_loc="0.0032004"/>
+    <create2_standoff_kinect parent="plate_2_link" number="1" x_loc="-0.1024382" y_loc="-0.098" z_loc="0.0032004"/>
+    <create2_standoff_8in parent="standoff_2in_4_link" number="0" x_loc="0" y_loc="0" z_loc="0.05715"/>
+    <create2_standoff_8in parent="standoff_2in_5_link" number="1" x_loc="0" y_loc="0" z_loc="0.05715"/>
+    <create2_standoff_8in parent="standoff_2in_6_link" number="2" x_loc="0" y_loc="0" z_loc="0.05715"/>
+    <create2_standoff_8in parent="standoff_2in_7_link" number="3" x_loc="0" y_loc="0" z_loc="0.05715"/>
     <joint name="plate_3_joint" type="fixed">
       <origin xyz="-0.01316 0 0.2063496" rpy="0 0 0" />
@@ -254,5 +254,5 @@
         <origin xyz=" 0 0 0 " rpy="0 0 0" />
         <geometry>
-          <mesh filename="package://turtlebot_description/meshes/stacks/circles/plate_2_logo.dae"/>
+          <mesh filename="package://create2_description/meshes/stacks/circles/plate_2_logo.dae"/>
         </geometry>
       </visual>
